File: pallas-ethernet-adapter.kicad_sch (KiCad schematic)
At the start: 25 parts, among them J3 PPS, J4 IE-CLK, J5 RJ45_LED_Shielded, J6 RESET, J7 JTAG

Commit message: * ground plane change to keep out beneath the magnetic module * changed RJ45 modular jack from tab up to tab down to improve the routing * added an 3d modell in the library folder for the rj45 connector * added a fitting footprint for SS74800-038F * changed width of the MDI and MII tracks to the JLC3313 stackup * changed impedance of the pcie lane from 100 Ohm differential to 85 Ohm and from 50 single ended to 45 ohm * impedace calculation pictures still missing
Parts:
- J5: footprint Connector_RJ:RJ45_Amphenol_RJHSE538X -> Library:SS74800038F; MPN SS-90000-009 -> SS74800-038F
Changed lines of the file:
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@@
     (property "Reference" "J5" (id 0) (at 231.14 29.21 0))
     (property "Value" "RJ45_LED_Shielded" (id 1) (at 231.14 31.75 0))
-    (property "Footprint" "Connector_RJ:RJ45_Amphenol_RJHSE538X" (id 2) (at 231.14 43.815 90)
-      (effects (font (size 1.27 1.27)) hide)
-    )
-    (property "Datasheet" "" (id 3) (at 231.14 43.815 90)
+    (property "Footprint" "Library:SS74800038F" (id 2) (at 231.14 43.815 90)
+      (effects (font (size 1.27 1.27)) hide)
+    )
+    (property "Datasheet" "https://www.mouser.de/datasheet/2/643/dr-STW-SS74800-038F-SS74800-087F-1570032.pdf" (id 3) (at 231.14 43.815 90)
       (effects (font (size 1.27 1.27)) hide)
     )
@@
       (effects (font (size 1.27 1.27)) hide)
     )
-    (property "MPN" "SS-90000-009" (id 5) (at 231.14 44.45 0)
+    (property "MPN" "SS74800-038F" (id 5) (at 231.14 44.45 0)
       (effects (font (size 1.27 1.27)) hide)
     )
@@
     )
     (path "/b570e801-bfe7-4a35-b59b-0f09030c449f"
-      (reference "J5") (unit 1) (value "RJ45_LED_Shielded") (footprint "Connector_RJ:RJ45_Amphenol_RJHSE538X")
+      (reference "J5") (unit 1) (value "RJ45_LED_Shielded") (footprint "Library:SS74800038F")
     )
     (path "/8d437fc2-b145-49df-a99a-ec4a1850a113"

Commit message: * removed R19 from jlcpcb CPL (PNP File) and from BOM fix: #2 * widened the holes for the RH45 connector by 0.1mm fix: #5 * added datasheets to documentation directory as well as a dummy graphic for the website
Other:
- note added: "Green"
- note added: "Orange"
Changed lines of the file:
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@@
     (stroke (width 0) (type default) (color 0 0 0 0))
+  )
+  (text "Orange" (at 242.57 35.56 0)
+    (effects (font (size 1.27 1.27)) (justify left bottom))
+  )
+  (text "Green" (at 242.57 50.8 0)
+    (effects (font (size 1.27 1.27)) (justify left bottom))
   )
   (label "LAN_JTAG_TDI" (at 166.37 85.09 180)
